File: Hardware/usb.kicad_sch (KiCad schematic)
At the start: 0 parts

Commit message: Completed schematic and PCB.
Parts:
- added C? (x2): 100n, Capacitor_SMD:C_0603_1608Metric_Pad1.08x0.95mm_HandSolder, symbol Device:C_Small
- added J?: DS1069-04MVW6X, symbol LVModule-rescue:Conn_01x04_Male-Connector
- added U?: ISO7221, Package_SO:SOIC-8_3.9x4.9mm_P1.27mm, symbol LVModule-rescue:ISO7221-oe_isolation
Connections:
- new net: C?.2, J?.4 (Pin_4), U?.5 (GND2)
- new net: J?.3 (Pin_3), U?.6 (OUT2)
- new net: J?.2 (Pin_2), U?.7 (IN2)
- new net: C?.1, J?.1 (Pin_1), U?.8 (VCC2)
- new net GND: C?.1, U?.4 (GND1)
- new net RX: U?.2 (OUT1)
- new net TX: U?.3 (IN1)
- new net VDD: C?.2, U?.1 (VCC1)
Changed lines of the file:
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@@
 (kicad_sch (version 20211123) (generator eeschema)
   (paper "A4")
+  (junction (at 129.54 91.44) (diameter 0) (color 0 0 0 0)
+  )
+  (junction (at 129.54 96.52) (diameter 0) (color 0 0 0 0)
+  )
+  (junction (at 153.035 101.6) (diameter 0) (color 0 0 0 0)
+  )
+  (junction (at 152.4 92.71) (diameter 0) (color 0 0 0 0)
+  )
+  (wire (pts (xy 151.765 102.87) (xy 151.765 99.06))
+    (stroke (width 0) (type solid) (color 0 0 0 0))
+  )
+  (wire (pts (xy 151.765 99.06) (xy 166.37 99.06))
+    (stroke (width 0) (type solid) (color 0 0 0 0))
+  )
+  (wire (pts (xy 129.54 91.44) (xy 128.27 91.44))
+    (stroke (width 0) (type solid) (color 0 0 0 0))
+  )
+  (wire (pts (xy 151.13 96.52) (xy 151.13 100.33))
+    (stroke (width 0) (type solid) (color 0 0 0 0))
+  )
+  (wire (pts (xy 129.54 95.25) (xy 129.54 96.52))
+    (stroke (width 0) (type solid) (color 0 0 0 0))
+  )
+  (wire (pts (xy 129.54 89.535) (xy 129.54 91.44))
+    (stroke (width 0) (type solid) (color 0 0 0 0))
+  )
+  (wire (pts (xy 129.54 92.71) (xy 129.54 91.44))
+    (stroke (width 0) (type solid) (color 0 0 0 0))
+  )
+  (wire (pts (xy 151.13 102.87) (xy 151.765 102.87))
+    (stroke (width 0) (type solid) (color 0 0 0 0))
+  )
+  (wire (pts (xy 166.37 93.98) (xy 152.4 93.98))
+    (stroke (width 0) (type solid) (color 0 0 0 0))
+  )
+  (wire (pts (xy 129.54 96.52) (xy 128.27 96.52))
+    (stroke (width 0) (type solid) (color 0 0 0 0))
+  )
+  (wire (pts (xy 152.4 92.075) (xy 152.4 92.71))
+    (stroke (width 0) (type solid) (color 0 0 0 0))
+  )
+  (wire (pts (xy 153.035 86.995) (xy 152.4 86.995))
+    (stroke (width 0) (type solid) (color 0 0 0 0))
+  )
+  (wire (pts (xy 153.035 101.6) (xy 152.4 101.6))
+    (stroke (width 0) (type solid) (color 0 0 0 0))
+  )
+  (wire (pts (xy 153.035 86.995) (xy 153.035 101.6))
+    (stroke (width 0) (type solid) (color 0 0 0 0))
+  )
+  (wire (pts (xy 130.81 92.71) (xy 129.54 92.71))
+    (stroke (width 0) (type solid) (color 0 0 0 0))
+  )
+  (wire (pts (xy 152.4 92.71) (xy 151.13 92.71))
+    (stroke (width 0) (type solid) (color 0 0 0 0))
+  )
+  (wire (pts (xy 166.37 101.6) (xy 153.035 101.6))
+    (stroke (width 0) (type solid) (color 0 0 0 0))
+  )
+  (wire (pts (xy 130.81 102.87) (xy 107.95 102.87))
+    (stroke (width 0) (type solid) (color 0 0 0 0))
+  )
+  (wire (pts (xy 129.54 96.52) (xy 129.54 104.775))
+    (stroke (width 0) (type default) (color 0 0 0 0))
+  )
+  (wire (pts (xy 151.13 96.52) (xy 166.37 96.52))
+    (stroke (width 0) (type solid) (color 0 0 0 0))
+  )
+  (wire (pts (xy 152.4 101.6) (xy 152.4 95.25))
+    (stroke (width 0) (type solid) (color 0 0 0 0))
+  )
+  (wire (pts (xy 130.81 100.33) (xy 107.95 100.33))
+    (stroke (width 0) (type solid) (color 0 0 0 0))
+  )
+  (wire (pts (xy 152.4 95.25) (xy 151.13 95.25))
+    (stroke (width 0) (type solid) (color 0 0 0 0))
+  )
+  (wire (pts (xy 152.4 93.98) (xy 152.4 92.71))
+    (stroke (width 0) (type solid) (color 0 0 0 0))
+  )
+  (wire (pts (xy 130.81 95.25) (xy 129.54 95.25))
+    (stroke (width 0) (type solid) (color 0 0 0 0))
+  )
+  (hierarchical_label "RX" (shape output) (at 107.95 100.33 180)
+    (effects (font (size 1.27 1.27)) (justify right))
+  )
+  (hierarchical_label "TX" (shape input) (at 107.95 102.87 180)
+    (effects (font (size 1.27 1.27)) (justify right))
+  )
+  (symbol (lib_id "Device:C_Small") (at 128.27 93.98 180) (unit 1)
+    (in_bom yes) (on_board yes)
+    (property "Reference" "C?" (id 0) (at 127 95.25 90)
+      (effects (font (size 1.27 1.27)) (justify left))
+    )
+    (property "Value" "100n" (id 1) (at 127 88.265 90)
+      (effects (font (size 1.27 1.27)) (justify left))
+    )
+    (property "Footprint" "Capacitor_SMD:C_0603_1608Metric_Pad1.08x0.95mm_HandSolder" (id 2) (at 128.27 93.98 0)
+      (effects (font (size 1.27 1.27)) hide)
+    )
+    (property "Datasheet" "~" (id 3) (at 128.27 93.98 0)
+      (effects (font (size 1.27 1.27)) hide)
+    )
+    (property "Link" "https://ozdisan.com/passive-components/capacitors/smt-smd-and-mlcc-capacitors/CL10B104KB8NNNC" (id 4) (at 128.27 93.98 0)
+      (effects (font (size 1.27 1.27)) hide)
+    )
+    (property "Price" "0.00448" (id 5) (at 128.27 93.98 0)
+      (effects (font (size 1.27 1.27)) hide)
+    )
+    (pin "1")
+    (pin "2")
+  )
+  (symbol (lib_id "power:GND") (at 129.54 104.775 0) (unit 1)
+    (in_bom yes) (on_board yes) (fields_autoplaced)
+    (property "Reference" "#PWR?" (id 0) (at 129.54 111.125 0)
+      (effects (font (size 1.27 1.27)) hide)
+    )
+    (property "Value" "GND" (id 1) (at 129.54 109.22 0))
+    (property "Footprint" "" (id 2) (at 129.54 104.775 0)
+      (effects (font (size 1.27 1.27)) hide)
+    )
+    (property "Datasheet" "" (id 3) (at 129.54 104.775 0)
+      (effects (font (size 1.27 1.27)) hide)
+    )
+    (pin "1")
+  )
+  (symbol (lib_id "power:VDD") (at 129.54 89.535 0) (unit 1)
+    (in_bom yes) (on_board yes) (fields_autoplaced)
+    (property "Reference" "#PWR?" (id 0) (at 129.54 93.345 0)
+      (effects (font (size 1.27 1.27)) hide)
+    )
+    (property "Value" "VDD" (id 1) (at 129.54 83.82 0))
+    (property "Footprint" "" (id 2) (at 129.54 89.535 0)
+      (effects (font (size 1.27 1.27)) hide)
+    )
+    (property "Datasheet" "" (id 3) (at 129.54 89.535 0)
+      (effects (font (size 1.27 1.27)) hide)
+    )
+    (pin "1")
+  )
+  (symbol (lib_id "LVModule-rescue:ISO7221-oe_isolation") (at 140.97 97.79 0) (unit 1)
+    (in_bom yes) (on_board yes)
+    (property "Reference" "U?" (id 0) (at 140.97 85.9282 0))
+    (property "Value" "ISO7221" (id 1) (at 140.97 88.2396 0))
+    (property "Footprint" "Package_SO:SOIC-8_3.9x4.9mm_P1.27mm" (id 2) (at 140.97 81.28 0)
+      (effects (font (size 1.27 1.27)) hide)
+    )
+    (property "Datasheet" "" (id 3) (at 140.97 81.28 0)
+      (effects (font (size 1.27 1.27)) hide)
+    )
+    (property "Link" "https://ozdisan.com/integrated-circuits-ics/interfaces-and-peripherals-ics/digital-isolators/ISO7221ADR" (id 4) (at 140.97 97.79 0)
+      (effects (font (size 1.27 1.27)) hide)
+    )
+    (property "Price" "4.9247" (id 5) (at 140.97 97.79 0)
+      (effects (font (size 1.27 1.27)) hide)
+    )
+    (pin "1")
+    (pin "2")
+    (pin "3")
+    (pin "4")
+    (pin "5")
+    (pin "6")
+    (pin "7")
+    (pin "8")
+  )
+  (symbol (lib_id "LVModule-rescue:Conn_01x04_Male-Connector") (at 171.45 96.52 0) (mirror y) (unit 1)
+    (in_bom yes) (on_board yes)
+    (property "Reference" "J?" (id 0) (at 172.1612 97.1804 0)
+      (effects (font (size 1.27 1.27)) (justify right))
+    )
+    (property "Value" "DS1069-04MVW6X" (id 1) (at 172.1612 99.4918 0)
+      (effects (font (size 1.27 1.27)) (justify right))
+    )
+    (property "Footprint" "" (id 2) (at 171.45 96.52 0)
+      (effects (font (size 1.27 1.27)) hide)
+    )
+    (property "Datasheet" "~" (id 3) (at 171.45 96.52 0)
+      (effects (font (size 1.27 1.27)) hide)
+    )
+    (property "Link" "https://ozdisan.com/connectors-and-interconnects/rectangular-connectors/pcb-connectors/DS1069-04MVW6X" (id 4) (at 171.45 96.52 0)
+      (effects (font (size 1.27 1.27)) hide)
+    )
+    (property "Price" "0.09086TL" (id 5) (at 171.45 96.52 0)
+      (effects (font (size 1.27 1.27)) hide)
+    )
+    (pin "1")
+    (pin "2")
+    (pin "3")
+    (pin "4")
+  )
+  (symbol (lib_id "Device:C_Small") (at 152.4 89.535 180) (unit 1)
+    (in_bom yes) (on_board yes)
+    (property "Reference" "C?" (id 0) (at 151.13 90.805 90)
+      (effects (font (size 1.27 1.27)) (justify left))
+    )
+    (property "Value" "100n" (id 1) (at 151.13 83.82 90)
+      (effects (font (size 1.27 1.27)) (justify left))
+    )
+    (property "Footprint" "Capacitor_SMD:C_0603_1608Metric_Pad1.08x0.95mm_HandSolder" (id 2) (at 152.4 89.535 0)
+      (effects (font (size 1.27 1.27)) hide)
+    )
+    (property "Datasheet" "~" (id 3) (at 152.4 89.535 0)
+      (effects (font (size 1.27 1.27)) hide)
+    )
+    (property "Link" "https://ozdisan.com/passive-components/capacitors/smt-smd-and-mlcc-capacitors/CL10B104KB8NNNC" (id 4) (at 152.4 89.535 0)
+      (effects (font (size 1.27 1.27)) hide)
+    )
+    (property "Price" "0.00448" (id 5) (at 152.4 89.535 0)
+      (effects (font (size 1.27 1.27)) hide)
+    )
+    (pin "1")
+    (pin "2")
+  )
 )
