File: Hardware/Wirebonder.kicad_sch (KiCad schematic)
At the start: 0 parts

Commit message: Completed schematic and PCB.
Other:
- sheet lever renamed zmotor
- sheet piezo renamed ultrasonic
- sheet usb renamed serial
- added sheet contact_sensors (contact_sensors.kicad_sch)
- added sheet drives (drives.kicad_sch)
- added sheet lvdt (lvdt.kicad_sch)
- added sheet regulators (regulators.kicad_sch)
- sheet force_coil ports: added ISENS, PWM, nPWM; removed none
- sheet interface ports: added INT, SCL, SDA; removed none
- sheet mcu ports: added CONTACT_SENSORS_MOUSE_LEFT, CONTACT_SENSORS_MOUSE_RIGHT, CONTACT_SENSORS_RES0, CONTACT_SENSORS_RES1, CONTACT_SENSORS_RES2, CONTACT_SENSORS_RES3, CONTACT_SENSORS_TIP, CONTACT_SENSORS_YLIM, DRIVES_AREALIGHT_nPWM, DRIVES_SOL1H, DRIVES_SOL1L, DRIVES_SOL2H, DRIVES_SOL2L, DRIVES_SOL3H, DRIVES_SOL3L, DRIVES_SPOTLIGHT_nPWM, FORCE_COIL_ISENS, FORCE_COIL_PWM, FORCE_COIL_nPWM, INTERFACE_INT, INTERFACE_SCL, INTERFACE_SDA, LVDT_A, LVDT_B, LVDT_SIGNAL, SERIAL_RX, SERIAL_TX, STEPPER_EN, STEPPER_FAULT, STEPPER_RESET, STEPPER_TEAR_DIR, STEPPER_TEAR_STEP, STEPPER_Y_DIR, STEPPER_Y_STEP, ULTRASONIC_ISENS, ULTRASONIC_SIGNAL, ULTRASONIC_VSENS, ZMOTOR_PWM, ZMOTOR_TACHOMETER, ZMOTOR_nPWM; removed none
- sheet serial: file usb.kicad_sch -> serial.kicad_sch
- sheet serial ports: added RX, TX; removed none
- sheet stepper ports: added EN, FAULT, RESET, TEAR_DIR, TEAR_STEP, Y_DIR, Y_STEP; removed none
- sheet ultrasonic: file piezo.kicad_sch -> ultrasonic.kicad_sch
- sheet ultrasonic ports: added ISENS, SIGNAL, VSENS; removed none
- sheet zmotor: file lever.kicad_sch -> zmotor.kicad_sch
- sheet zmotor ports: added PWM, TACHOMETER, nPWM; removed none
