File: Hardware/interface.kicad_sch (KiCad schematic)
At the start: 0 parts

Commit message: Completed schematic and PCB.
Parts:
- added C68, C69: 100n, Capacitor_SMD:C_0603_1608Metric_Pad1.08x0.95mm_HandSolder, symbol Device:C_Small
- added J10: DS1021-1X14SF11-B, Connector_PinHeader_2.54mm:PinHeader_1x14_P2.54mm_Vertical, symbol Connector:Conn_01x14_Male
- added J8: Conn_02x07_Odd_Even, Connector_IDC:IDC-Header_2x07_P2.54mm_Vertical, symbol Connector_Generic:Conn_02x07_Odd_Even
- added J9: Conn_02x08_Odd_Even, Connector_IDC:IDC-Header_2x08_P2.54mm_Vertical, symbol Connector_Generic:Conn_02x08_Odd_Even
- added Q15, Q16, Q17, Q18: BC807-40, Package_TO_SOT_SMD:SOT-23, symbol Device:Q_PNP_BEC
- added Q19: BC817-40, Package_TO_SOT_SMD:SOT-23, symbol Transistor_BJT:BC817
- added R100, R101, R102, R103, R104, R107, R109, R110, R111, R112, R78, R84, R85, R86, R87, R88, R89, R94, R95, R96, R97, R98, R99: 10k, Resistor_SMD:R_0603_1608Metric_Pad0.98x0.95mm_HandSolder, symbol Device:R_Small
- added R108: 1k, Resistor_SMD:R_0603_1608Metric_Pad0.98x0.95mm_HandSolder, symbol Device:R_Small
- added R113: 4.7k, Resistor_SMD:R_0603_1608Metric_Pad0.98x0.95mm_HandSolder, symbol Device:R_Small
- added R76, R77: 2.2k, Resistor_SMD:R_0603_1608Metric_Pad0.98x0.95mm_HandSolder, symbol Device:R_Small
- added R79, R80, R81, R82, R83: 0R, Resistor_SMD:R_0603_1608Metric_Pad0.98x0.95mm_HandSolder, symbol Device:R_Small
- added R90, R91, R92, R93: 470R, Resistor_SMD:R_0603_1608Metric_Pad0.98x0.95mm_HandSolder, symbol Device:R_Small
- added RV1: 10k, Potentiometer_SMD:Potentiometer_Bourns_3314G_Vertical, symbol Device:R_Potentiometer
- added U12: PCA9535, Package_SO:QSOP-24_3.9x8.7mm_P0.635mm, symbol expander:PCA9535
- added U13: PCA9538, Package_SO:TSSOP-16_4.4x5mm_P0.65mm, symbol expander:PCA9538
Connections:
- new net: Q17.3 (C), R103.2, U12.15 (IO1_2)
- new net: R83.1, R89.1, U13.2 (A1)
- new net: J10.8 (Pin_8), R110.1
- new net: Q15.3 (C), R101.2, U12.13 (IO1_0)
- new net: Q15.2 (E), Q16.2 (E), Q17.2 (E), Q18.2 (E), Q19.2 (E), R107.1
- new net: J8.8 (Pin_8), R94.2, U12.4 (IO0_0)
- new net: J8.1 (Pin_1), J9.3 (Pin_3), R100.2, U12.10 (IO0_6)
- new net: Q16.3 (C), R102.2, U12.14 (IO1_1)
- new net: Q18.3 (C), R104.2, U12.16 (IO1_3)
- new net: R90.1, U12.17 (IO1_4)
- new net: R91.1, U12.18 (IO1_5)
- new net: R92.1, U12.19 (IO1_6)
- new net: R80.1, R86.1, U12.2 (A1)
- new net: R93.1, U12.20 (IO1_7)
- new net: R79.1, R85.1, U12.21 (A0)
- new net: R81.1, R88.1, U12.3 (A2)
- new net: J8.7 (Pin_7), R95.2, U12.5 (IO0_1)
- new net: J8.6 (Pin_6), J9.8 (Pin_8), R96.2, U12.6 (IO0_2)
- new net: J8.5 (Pin_5), J9.7 (Pin_7), R97.2, U12.7 (IO0_3)
- new net: J8.4 (Pin_4), J9.6 (Pin_6), R98.2, U12.8 (IO0_4)
- new net: J8.3 (Pin_3), J9.5 (Pin_5), R99.2, U12.9 (IO0_5)
- new net: J8.13 (Pin_13), Q16.1 (B)
- new net: J10.10 (Pin_10), R112.1
- new net: J10.3 (Pin_3), RV1.2
- new net: J10.7 (Pin_7), R109.1
- new net: J10.9 (Pin_9), R111.1
- new net: R84.2, U13.3 (~{RESET})
- new net: J9.10 (Pin_10), R90.2
- new net: Q19.1 (B), R108.2, R113.1
- new net: J9.11 (Pin_11), R92.2
- new net: J8.11 (Pin_11), Q15.1 (B)
- new net: R82.1, R87.1, U13.1 (A0)
- new net: J9.14 (Pin_14), Q18.1 (B)
- new net: J8.14 (Pin_14), Q17.1 (B)
- new net: J9.12 (Pin_12), R91.2
- new net: J8.9 (Pin_9), R93.2
- new net +5V: J10.2 (Pin_2), Q19.3 (C), R108.1, RV1.1
- new net D4: J10.11 (Pin_11), U13.7 (P3)
- new net D5: J10.12 (Pin_12), U13.9 (P4)
- new net D6: J10.13 (Pin_13), U13.10 (P5)
- new net D7: J10.14 (Pin_14), U13.11 (P6)
- new net EN: J10.6 (Pin_6), U13.6 (P2)
- new net GND: C68.2, C69.1, J10.1 (Pin_1), J8.2 (Pin_2), J9.2 (Pin_2), R100.1, R101.1, R102.1, R103.1, R104.1, R107.2, R109.2, R110.2, R111.2, R112.2, R113.2, R85.2, R86.2, R87.2, R88.2, R89.2, R94.1, R95.1, R96.1, R97.1, R98.1, R99.1, RV1.3, U12.12 (VSS), U13.8 (VSS)
- new net INT: R78.2, U12.1 (~{INT})
- new net RS: J10.4 (Pin_4), U13.4 (P0)
- new net RW: J10.5 (Pin_5), U13.5 (P1)
- new net SCL: R76.1, U12.22 (SCL), U13.14 (SCL)
- new net SDA: R77.1, U12.23 (SDA), U13.15 (SDA)
- new net VDD: C68.1, C69.2, R76.2, R77.2, R78.1, R79.2, R80.2, R81.2, R82.2, R83.2, R84.1, U12.24 (VCC), U13.16 (VCC)
- no-connect marks 0 -> 11
