File: Hardware/mcu.kicad_sch (KiCad schematic)
At the start: 1 part

Commit message: Completed schematic and PCB.
Parts:
- removed U?: STM32G431CBTx, Package_QFP:LQFP-48_7x7mm_P0.5mm, symbol LibreSolar:STM32G431CBTx
- added C11, C12: 18p, Capacitor_SMD:C_0603_1608Metric_Pad1.08x0.95mm_HandSolder, symbol Device:C_Small
- added C13, C16, C17, C18, C19, C21, C23: 100n, Capacitor_SMD:C_0603_1608Metric_Pad1.08x0.95mm_HandSolder, symbol Device:C_Small
- added C14: 4.7u, Capacitor_SMD:C_0603_1608Metric_Pad1.08x0.95mm_HandSolder, symbol Device:C_Small
- added C15, C20: 1u, Capacitor_SMD:C_0603_1608Metric_Pad1.08x0.95mm_HandSolder, symbol Device:C_Small
- added J3: Conn_02x05_Odd_Even, Connector_PinHeader_2.54mm:PinHeader_2x05_P2.54mm_Vertical, symbol Connector_Generic:Conn_02x05_Odd_Even
- added R22: 10k, Resistor_SMD:R_0603_1608Metric_Pad0.98x0.95mm_HandSolder, symbol Device:R_Small
- added U3: STM32F446RCTx, Package_QFP:LQFP-64_10x10mm_P0.5mm, symbol MCU_ST_STM32F4:STM32F446RCTx
- added Y1: 8MHz 85ohms, Crystal:Crystal_SMD_5032-4Pin_5.0x3.2mm, symbol Device:Crystal_GND24
Connections:
- net GND: now also C11.1, C12.1, C13.1, C14.2, C15.1, C16.1, C17.1, C18.1, C19.1, C20.2, C21.2, C23.1, J3.9 (Pin_9), R22.2, U3.12 (VSSA), U3.18 (VSS), U3.31 (VSS), U3.47 (VSS), U3.63 (VSS), Y1.2, Y1.4
- new net: C12.2, U3.6 (PH1), Y1.1
- new net: C11.2, U3.5 (PH0), Y1.3
- new net: R22.1, U3.60 (BOOT0)
- new net: C15.2, U3.1 (VBAT)
- new net: C14.1, U3.30 (VCAP_1)
- new net CONTACT_SENSORS_MOUSE_LEFT: U3.11 (PC3)
- new net CONTACT_SENSORS_MOUSE_RIGHT: U3.10 (PC2)
- new net CONTACT_SENSORS_RES0: U3.62 (PB9)
- new net CONTACT_SENSORS_RES1: U3.2 (PC13)
- new net CONTACT_SENSORS_RES2: U3.3 (PC14)
- new net CONTACT_SENSORS_RES3: U3.4 (PC15)
- new net CONTACT_SENSORS_TIP: U3.8 (PC0)
- new net CONTACT_SENSORS_YLIM: U3.9 (PC1)
- new net DRIVES_AREALIGHT_nPWM: U3.37 (PC6)
- new net DRIVES_SOL1H: U3.24 (PC4)
- new net DRIVES_SOL1L: U3.26 (PB0)
- new net DRIVES_SOL2H: U3.27 (PB1)
- new net DRIVES_SOL2L: U3.28 (PB2)
- new net DRIVES_SOL3H: U3.36 (PB15)
- new net DRIVES_SOL3L: U3.33 (PB12)
- new net DRIVES_SPOTLIGHT_nPWM: U3.38 (PC7)
- new net FORCE_COIL_ISENS: U3.16 (PA2)
- new net FORCE_COIL_PWM: U3.41 (PA8)
- new net FORCE_COIL_nPWM: U3.34 (PB13)
- new net INTERFACE_INT: U3.57 (PB5)
- new net INTERFACE_SCL: U3.58 (PB6)
- new net INTERFACE_SDA: U3.59 (PB7)
- new net LVDT_A: U3.22 (PA6)
- new net LVDT_B: U3.23 (PA7)
- new net LVDT_SIGNAL: U3.21 (PA5)
- new net NRST: C13.2, J3.3 (Pin_3), U3.7 (NRST)
- new net PB3: J3.2 (Pin_2), U3.55 (PB3)
- new net PB4: J3.4 (Pin_4), U3.56 (PB4)
- new net PB8: J3.6 (Pin_6), U3.61 (PB8)
- new net PC11: J3.8 (Pin_8), U3.52 (PC11)
- new net PC12: J3.10 (Pin_10), U3.53 (PC12)
- new net SERIAL_RX: U3.25 (PC5)
- new net SERIAL_TX: U3.29 (PB10)
- new net STEPPER_EN: U3.45 (PA12)
- new net STEPPER_FAULT: U3.50 (PA15)
- new net STEPPER_RESET: U3.51 (PC10)
- new net STEPPER_TEAR_DIR: U3.40 (PC9)
- new net STEPPER_TEAR_STEP: U3.39 (PC8)
- new net STEPPER_Y_DIR: U3.44 (PA11)
- new net STEPPER_Y_STEP: U3.43 (PA10)
- new net SWCLK: J3.5 (Pin_5), U3.49 (PA14)
- new net SWDIO: J3.7 (Pin_7), U3.46 (PA13)
- new net ULTRASONIC_ISENS: U3.15 (PA1)
- new net ULTRASONIC_SIGNAL: U3.20 (PA4)
- new net ULTRASONIC_VSENS: U3.14 (PA0)
- new net VDD: C16.2, C17.2, C18.2, C19.2, C23.2, J3.1 (Pin_1), U3.19 (VDD), U3.32 (VDD), U3.48 (VDD), U3.64 (VDD)
- new net VDDA: C20.1, C21.1, U3.13 (VDDA)
- new net ZMOTOR_PWM: U3.42 (PA9)
- new net ZMOTOR_TACHOMETER: U3.17 (PA3)
- new net ZMOTOR_nPWM: U3.35 (PB14)
- no-connect marks 0 -> 1

Commit message: Few coonector footprint modifications and silkscreen additions to them.
Parts:
- J3: Link (none) -> https://ozdisan.com/connectors-and-interconnects/headers/pi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; Price (none) -> 0.04014
Changed lines of the file:
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@@
+      (effects (font (size 1.27 1.27)) hide)
+    )
+    (property "Link" "https://ozdisan.com/connectors-and-interconnects/headers/pin-headers/L-KLS1-207-2-10-S" (id 4) (at 239.395 39.37 0)
+      (effects (font (size 1.27 1.27)) hide)
+    )
+    (property "Price" "0.04014" (id 5) (at 239.395 39.37 0)
       (effects (font (size 1.27 1.27)) hide)
     )
