File: Hardware/ultrasonic.kicad_sch (KiCad schematic)
At the start: 74 parts, among them J4 DG250-3-5-02P-11-00AH, Q1 BC817-40, Q2 BC817-40, Q3 BCP53-16, Q4 BCP56-16, Q5 BCP53-16, Q6 BCP56-16, Q7 MJD45H11T4G, Q8 MJD44H11T4G, U4 AD8656, U5 AD8656

Commit message: Snapshot: C++ firmware refactor + debugBridge tooling + PWM/nPWM fixes
Working-state backup of the ongoing rewrite:
- Firmware ported to modular C++ (services / modules / debug channels);
  legacy C modules removed.
- Multi-controller (bool-return) callback mechanism across signal channels.
- debugBridge GDB test package (DebugService protocol) added.
- TIM1 complementary (nPWM) outputs enabled + 500 ns dead-time for the
  IRS2005 half-bridges.
- Vendored STM32 HAL drivers + host GoogleTest sources; .gitignore for
  build/cache artifacts.
- Includes Hardware schematic and Scripts updates present in the tree.
Parts:
- Q7: value MJD45H11T4G -> MJD44H11T4G
- Q8: value MJD44H11T4G -> MJD45H11T4G
